File: pcb/tes1.brd (EAGLE design)
At the start: 100 x 80 mm, 28 parts, among them IC1 MEGA8-AI, T1 MJD31, T2 MJD31

Commit message: ready to manufactured
Parts:
- removed ISP-B1: 1x3 RA Female .1", SparkFun-Connectors:1X03_SMD_RA_FEMALE
- added ISP-A, UART: 1x3 RA Female .1", SparkFun-Connectors:1X03_SMD_RA_FEMALE
- JP2: value USB-B-S -> (none); device SparkFun-Connectors:USB-B-SMT -> con-berg:PN87520
- moved JP2 143.0 mm to (79.5, 12.2), flipped to the bottom, turned to 270 degrees
- moved LED4 126.5 mm to (42.5, 51.7), flipped to the bottom, turned to 270 degrees
- moved LED3 121.2 mm to (38.7, 51.7), flipped to the bottom, turned to 270 degrees
- moved R6 119.6 mm to (59.2, 18.0), flipped to the bottom, turned to 90 degrees
- moved D5 118.2 mm to (70.9, 15.4), flipped to the bottom, turned to 90 degrees
- moved LED2 116.0 mm to (34.9, 51.7), flipped to the bottom, turned to 270 degrees
- moved LED1 110.8 mm to (31.1, 51.7), flipped to the bottom, turned to 270 degrees
- moved D4 105.0 mm to (64.4, 5.84), flipped to the bottom
- moved R5 98.2 mm to (42.7, 11.9), flipped to the bottom, turned to 90 degrees
- moved T2 98.1 mm to (63.9, 15.0), flipped to the bottom, turned to 180 degrees
- moved C3 96.7 mm to (53.5, 9.91), flipped to the bottom, turned to 270 degrees
- moved R4 91.7 mm to (40.1, 11.9), flipped to the bottom, turned to 90 degrees
- moved R1 84.3 mm to (25.4, 14.9), flipped to the bottom, turned to 90 degrees
- moved IC1 83.2 mm to (35.2, 39.6), flipped to the bottom, turned to 270 degrees
- moved L1 81.7 mm to (40.1, 28.1), flipped to the bottom, turned to 180 degrees
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Connections:
- new net N$20: IC1.31, UART.2
- new net N$21: IC1.30, UART.1
- net CONVIN: now also IC1.27; no longer IC1.26
- net CONVOUT: now also IC1.26; no longer IC1.27
- net GND: now also ISP-A.2, JP2.4, UART.3; no longer ISP-B1.2, JP2.GND
- net N$12: now also ISP-A.3; no longer ISP-B1.3
- net N$16: now also IC1.9; no longer IC1.1
- net N$17: now also IC1.2; no longer IC1.32
- net N$18: now also IC1.1; no longer IC1.31
- net N$19: now also IC1.32; no longer IC1.30
- net VBATT: now also IC1.23; no longer IC1.24
- net VCC1: now also IC1.24; no longer IC1.23
- net VCC2: now also ISP-A.1; no longer ISP-B1.1
- net VCC3: now also JP2.1; no longer JP2.VUSB
Routing:
- net GND: track 0.00 -> 295.1 mm
- net VCC2: track 0.00 -> 114.9 mm, vias 0 -> 2
- net CONVOUT: track 0.00 -> 86.8 mm, vias 0 -> 2
- net VCC3: track 0.00 -> 70.8 mm, vias 0 -> 2
- net VBATT: track 0.00 -> 59.6 mm
- net VCC1: track 0.00 -> 58.4 mm
- net CONVIN: track 0.00 -> 27.9 mm
- net N$4: track 0.00 -> 15.7 mm
- net N$9: track 0.00 -> 13.1 mm
- net N$21: track 0.00 -> 12.5 mm
- net N$8: track 0.00 -> 10.9 mm
- net N$17: track 0.00 -> 10.0 mm
- net N$20: track 0.00 -> 9.52 mm
- net N$16: track 0.00 -> 9.48 mm
- net N$7: track 0.00 -> 8.41 mm
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- added copper zone on layer 16, net GND
Other:
- board size 100 x 80 mm -> 81.7 x 55.9 mm
