File: pcb/tes1.sch (EAGLE design)
At the start: 28 parts, among them IC1 MEGA8-AI, T1 MJD31, T2 MJD31

Commit message: ready to manufactured
Parts:
- added UART: 1x3 RA Female .1", SparkFun-Connectors:M03SMD_RA_FEMALE
- JP2: value USB-B-S -> (none); device SparkFun-Connectors:USB-B-S -> con-berg:PN87520
- renumbered ISP-B1 to ISP-A
Connections:
- new net N$20: IC1.PD1(TXD), UART.2
- new net N$21: IC1.PD0(RXD), UART.1
- net CONVIN: now also IC1.PC4(ADC4/SDA); no longer IC1.PC3(ADC3)
- net CONVOUT: now also IC1.PC3(ADC3); no longer IC1.PC4(ADC4/SDA)
- net GND: now also JP2.4, UART.3; no longer JP2.GND
- net N$16: now also IC1.PD5(T1); no longer IC1.PD3(INT1)
- net N$17: now also IC1.PD4(XCK/T0); no longer IC1.PD2(INT0)
- net N$18: now also IC1.PD3(INT1); no longer IC1.PD1(TXD)
- net N$19: now also IC1.PD2(INT0); no longer IC1.PD0(RXD)
- net VBATT: now also IC1.PC0(ADC0); no longer IC1.PC1(ADC1)
- net VCC1: now also IC1.PC1(ADC1); no longer IC1.PC0(ADC0)
- net VCC3: now also JP2.1; no longer JP2.VBUS
Other:
- moved on the sheet: JP2, LED1, LED2, LED3, LED4
Changed lines of the file:
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@@
 <part name="R7" library="rcl" deviceset="R-EU_" device="R1206" value="4k7"/>
 <part name="ISP-B" library="SparkFun-Connectors" deviceset="M03" device="SMD_RA_FEMALE" value="1x3 RA Female .1&quot;"/>
-<part name="ISP-B1" library="SparkFun-Connectors" deviceset="M03" device="SMD_RA_FEMALE" value="1x3 RA Female .1&quot;"/>
+<part name="ISP-A" library="SparkFun-Connectors" deviceset="M03" device="SMD_RA_FEMALE" value="1x3 RA Female .1&quot;"/>
 <part name="LED1" library="led" deviceset="LED" device="SML1206"/>
 <part name="LED2" library="led" deviceset="LED" device="SML1206"/>
 <part name="LED3" library="led" deviceset="LED" device="SML1206"/>
 <part name="LED4" library="led" deviceset="LED" device="SML1206"/>
-<part name="JP2" library="SparkFun-Connectors" deviceset="USB" device="-B-S"/>
+<part name="JP2" library="con-berg" deviceset="PN87520" device=""/>
+<part name="UART" library="SparkFun-Connectors" deviceset="M03" device="SMD_RA_FEMALE" value="1x3 RA Female .1&quot;"/>
 </parts>
 <sheets>
@@
 <instance part="R7" gate="G$1" x="83.82" y="2.54"/>
 <instance part="ISP-B" gate="G$1" x="152.4" y="-53.34" rot="R180"/>
-<instance part="ISP-B1" gate="G$1" x="104.14" y="12.7" rot="R180"/>
-<instance part="LED1" gate="G$1" x="144.78" y="-20.32" rot="R90"/>
-<instance part="LED2" gate="G$1" x="144.78" y="-22.86" rot="R90"/>
-<instance part="LED3" gate="G$1" x="144.78" y="-25.4" rot="R90"/>
-<instance part="LED4" gate="G$1" x="144.78" y="-27.94" rot="R90"/>
+<instance part="ISP-A" gate="G$1" x="104.14" y="12.7" rot="R180"/>
+<instance part="LED1" gate="G$1" x="144.78" y="-25.4" rot="R90"/>
+<instance part="LED2" gate="G$1" x="144.78" y="-27.94" rot="R90"/>
+<instance part="LED3" gate="G$1" x="144.78" y="-30.48" rot="R90"/>
+<instance part="LED4" gate="G$1" x="144.78" y="-33.02" rot="R90"/>
 <instance part="JP2" gate="G$1" x="35.56" y="-33.02"/>
+<instance part="UART" gate="G$1" x="170.18" y="-22.86" rot="R180"/>
 </instances>
 <busses>
@@
 </segment>
 <segment>
-<pinref part="IC1" gate="G$1" pin="PC0(ADC0)"/>
-<wire x1="139.7" y1="2.54" x2="147.32" y2="2.54" width="0.1524" layer="91"/>
-<label x="147.32" y="2.54" size="1.778" layer="95"/>
+<pinref part="IC1" gate="G$1" pin="PC1(ADC1)"/>
+<wire x1="139.7" y1="0" x2="147.32" y2="0" width="0.1524" layer="91"/>
+<label x="147.32" y="0" size="1.778" layer="95"/>
 </segment>
 </net>
@@
 </segment>
 <segment>
-<pinref part="ISP-B1" gate="G$1" pin="2"/>
+<pinref part="ISP-A" gate="G$1" pin="2"/>
 <wire x1="96.52" y1="12.7" x2="91.44" y2="12.7" width="0.1524" layer="91"/>
 <label x="83.82" y="12.7" size="1.778" layer="95"/>
@@
 <segment>
 <pinref part="LED1" gate="G$1" pin="C"/>
-<wire x1="149.86" y1="-20.32" x2="154.94" y2="-20.32" width="0.1524" layer="91"/>
-<wire x1="154.94" y1="-20.32" x2="154.94" y2="-22.86" width="0.1524" layer="91"/>
+<wire x1="149.86" y1="-25.4" x2="154.94" y2="-25.4" width="0.1524" layer="91"/>
+<wire x1="154.94" y1="-25.4" x2="154.94" y2="-27.94" width="0.1524" layer="91"/>
 <pinref part="LED4" gate="G$1" pin="C"/>
-<wire x1="154.94" y1="-22.86" x2="154.94" y2="-25.4" width="0.1524" layer="91"/>
-<wire x1="154.94" y1="-25.4" x2="154.94" y2="-27.94" width="0.1524" layer="91"/>
-<wire x1="154.94" y1="-27.94" x2="149.86" y2="-27.94" width="0.1524" layer="91"/>
+<wire x1="154.94" y1="-27.94" x2="154.94" y2="-30.48" width="0.1524" layer="91"/>
+<wire x1="154.94" y1="-30.48" x2="154.94" y2="-33.02" width="0.1524" layer="91"/>
+<wire x1="154.94" y1="-33.02" x2="149.86" y2="-33.02" width="0.1524" layer="91"/>
 <pinref part="LED3" gate="G$1" pin="C"/>
-<wire x1="149.86" y1="-25.4" x2="154.94" y2="-25.4" width="0.1524" layer="91"/>
+<wire x1="149.86" y1="-30.48" x2="154.94" y2="-30.48" width="0.1524" layer="91"/>
 <pinref part="LED2" gate="G$1" pin="C"/>
-<wire x1="149.86" y1="-22.86" x2="154.94" y2="-22.86" width="0.1524" layer="91"/>
-<label x="154.94" y="-27.94" size="1.778" layer="95"/>
-</segment>
-<segment>
-<pinref part="JP2" gate="G$1" pin="GND"/>
-<wire x1="33.02" y1="-33.02" x2="25.4" y2="-33.02" width="0.1524" layer="91"/>
-<label x="17.78" y="-33.02" size="1.778" layer="95"/>
+<wire x1="149.86" y1="-27.94" x2="154.94" y2="-27.94" width="0.1524" layer="91"/>
+<label x="154.94" y="-33.02" size="1.778" layer="95"/>
+<pinref part="UART" gate="G$1" pin="3"/>
+<wire x1="162.56" y1="-25.4" x2="154.94" y2="-25.4" width="0.1524" layer="91"/>
+</segment>
+<segment>
+<pinref part="JP2" gate="G$1" pin="4"/>
+<wire x1="33.02" y1="-35.56" x2="25.4" y2="-35.56" width="0.1524" layer="91"/>
+<label x="22.86" y="-35.56" size="1.778" layer="95"/>
 </segment>
 </net>
@@
 </segment>
 <segment>
-<pinref part="IC1" gate="G$1" pin="PC1(ADC1)"/>
-<wire x1="139.7" y1="0" x2="147.32" y2="0" width="0.1524" layer="91"/>
-<label x="147.32" y="0" size="1.778" layer="95"/>
+<pinref part="IC1" gate="G$1" pin="PC0(ADC0)"/>
+<wire x1="139.7" y1="2.54" x2="147.32" y2="2.54" width="0.1524" layer="91"/>
+<label x="147.32" y="2.54" size="1.778" layer="95"/>
 </segment>
 </net>
@@
 </segment>
 <segment>
-<pinref part="IC1" gate="G$1" pin="PC3(ADC3)"/>
-<wire x1="139.7" y1="-5.08" x2="147.32" y2="-5.08" width="0.1524" layer="91"/>
-<label x="147.32" y="-5.08" size="1.778" layer="95"/>
+<pinref part="IC1" gate="G$1" pin="PC4(ADC4/SDA)"/>
+<wire x1="139.7" y1="-7.62" x2="147.32" y2="-7.62" width="0.1524" layer="91"/>
+<label x="147.32" y="-7.62" size="1.778" layer="95"/>
 </segment>
 </net>
@@
 </segment>
 <segment>
-<pinref part="ISP-B1" gate="G$1" pin="1"/>
+<pinref part="ISP-A" gate="G$1" pin="1"/>
 <wire x1="96.52" y1="15.24" x2="91.44" y2="15.24" width="0.1524" layer="91"/>
 <label x="83.82" y="15.24" size="1.778" layer="95"/>
@@
 </segment>
 <segment>
-<pinref part="JP2" gate="G$1" pin="VBUS"/>
-<wire x1="33.02" y1="-30.48" x2="25.4" y2="-30.48" width="0.1524" layer="91"/>
-<label x="17.78" y="-30.48" size="1.778" layer="95"/>
+<pinref part="JP2" gate="G$1" pin="1"/>
+<wire x1="33.02" y1="-27.94" x2="25.4" y2="-27.94" width="0.1524" layer="91"/>
+<label x="22.86" y="-27.94" size="1.778" layer="95"/>
 </segment>
 </net>
@@
 </segment>
 <segment>
-<pinref part="IC1" gate="G$1" pin="PC4(ADC4/SDA)"/>
-<wire x1="139.7" y1="-7.62" x2="147.32" y2="-7.62" width="0.1524" layer="91"/>
-<label x="147.32" y="-7.62" size="1.778" layer="95"/>
+<pinref part="IC1" gate="G$1" pin="PC3(ADC3)"/>
+<wire x1="139.7" y1="-5.08" x2="147.32" y2="-5.08" width="0.1524" layer="91"/>
+<label x="147.32" y="-5.08" size="1.778" layer="95"/>
 </segment>
 </net>
@@
 <pinref part="R7" gate="G$1" pin="2"/>
 <wire x1="91.44" y1="2.54" x2="88.9" y2="2.54" width="0.1524" layer="91"/>
-<pinref part="ISP-B1" gate="G$1" pin="3"/>
+<pinref part="ISP-A" gate="G$1" pin="3"/>
 <wire x1="96.52" y1="10.16" x2="91.44" y2="10.16" width="0.1524" layer="91"/>
 <wire x1="91.44" y1="10.16" x2="91.44" y2="2.54" width="0.1524" layer="91"/>
@@
 <net name="N$16" class="0">
 <segment>
+<pinref part="IC1" gate="G$1" pin="PD5(T1)"/>
 <pinref part="LED4" gate="G$1" pin="A"/>
+<wire x1="139.7" y1="-33.02" x2="142.24" y2="-33.02" width="0.1524" layer="91"/>
+</segment>
+</net>
+<net name="N$17" class="0">
+<segment>
+<pinref part="IC1" gate="G$1" pin="PD4(XCK/T0)"/>
+<pinref part="LED3" gate="G$1" pin="A"/>
+<wire x1="139.7" y1="-30.48" x2="142.24" y2="-30.48" width="0.1524" layer="91"/>
+</segment>
+</net>
+<net name="N$18" class="0">
+<segment>
 <pinref part="IC1" gate="G$1" pin="PD3(INT1)"/>
-<wire x1="142.24" y1="-27.94" x2="139.7" y2="-27.94" width="0.1524" layer="91"/>
-</segment>
-</net>
-<net name="N$17" class="0">
-<segment>
-<pinref part="LED3" gate="G$1" pin="A"/>
+<pinref part="LED2" gate="G$1" pin="A"/>
+<wire x1="139.7" y1="-27.94" x2="142.24" y2="-27.94" width="0.1524" layer="91"/>
+</segment>
+</net>
+<net name="N$19" class="0">
+<segment>
 <pinref part="IC1" gate="G$1" pin="PD2(INT0)"/>
-<wire x1="142.24" y1="-25.4" x2="139.7" y2="-25.4" width="0.1524" layer="91"/>
-</segment>
-</net>
-<net name="N$18" class="0">
-<segment>
-<pinref part="LED2" gate="G$1" pin="A"/>
+<pinref part="LED1" gate="G$1" pin="A"/>
+<wire x1="139.7" y1="-25.4" x2="142.24" y2="-25.4" width="0.1524" layer="91"/>
+</segment>
+</net>
+<net name="N$20" class="0">
+<segment>
 <pinref part="IC1" gate="G$1" pin="PD1(TXD)"/>
-<wire x1="142.24" y1="-22.86" x2="139.7" y2="-22.86" width="0.1524" layer="91"/>
-</segment>
-</net>
-<net name="N$19" class="0">
-<segment>
-<pinref part="LED1" gate="G$1" pin="A"/>
+<pinref part="UART" gate="G$1" pin="2"/>
+<wire x1="139.7" y1="-22.86" x2="162.56" y2="-22.86" width="0.1524" layer="91"/>
+</segment>
+</net>
+<net name="N$21" class="0">
+<segment>
 <pinref part="IC1" gate="G$1" pin="PD0(RXD)"/>
-<wire x1="142.24" y1="-20.32" x2="139.7" y2="-20.32" width="0.1524" layer="91"/>
-</segment>
-</net>
+<pinref part="UART" gate="G$1" pin="1"/>
+<wire x1="139.7" y1="-20.32" x2="162.56" y2="-20.32" width="0.1524" layer="91"/>
+</segment>
+</net>
